Commit message: Update joint name

File: cnoid_tank_description/urdf/track.urdf.xacro (robot description, xacro)
@@ -3,5 +3,12 @@
   <xacro:include filename="$(find cnoid_tank_description)/urdf/common.xacro"/>
   <xacro:macro name="cnoid_tank_track" params="suffix side">
-    <link name="TRACK_${suffix}">
+    <link name="TRACK_${suffix}"/>
+    <joint name="TRACK_${suffix}" type="continuous">
+      <axis xyz="0 ${side} 0"/>
+      <origin xyz="0 ${side * 0.22} -0.026"/>
+      <parent link="CHASSIS"/>
+      <child link="TRACK_${suffix}"/>
+    </joint>
+    <link name="BELT_${suffix}">
       <visual>
         <geometry>
@@ -15,8 +22,8 @@
       </collision>
     </link>
-    <joint name="TRACK_${suffix}" type="fixed">
+    <joint name="BELT_${suffix}" type="fixed">
       <origin xyz="0 ${side * 0.22} -0.026"/>
       <parent link="CHASSIS"/>
-      <child link="TRACK_${suffix}"/>
+      <child link="BELT_${suffix}"/>
     </joint>
     <link name="WHEEL_${suffix}0">
@@ -34,5 +41,5 @@
     <joint name="WHEEL_${suffix}0" type="fixed">
       <origin xyz="0.25 ${side * -0.005} 0"/>
-      <parent link="TRACK_${suffix}"/>
+      <parent link="BELT_${suffix}"/>
       <child link="WHEEL_${suffix}0"/>
     </joint>
@@ -51,5 +58,5 @@
     <joint name="WHEEL_${suffix}1" type="fixed">
       <origin xyz="0 ${side * -0.005} 0"/>
-      <parent link="TRACK_${suffix}"/>
+      <parent link="BELT_${suffix}"/>
       <child link="WHEEL_${suffix}1"/>
     </joint>
@@ -68,5 +75,5 @@
     <joint name="WHEEL_${suffix}2" type="fixed">
       <origin xyz="-0.25 ${side * -0.005} 0"/>
-      <parent link="TRACK_${suffix}"/>
+      <parent link="BELT_${suffix}"/>
       <child link="WHEEL_${suffix}2"/>
     </joint>
