Commit message: Fix for choreonoid_ros update
* Use PointCloud2 instead of PointCloud
* Fix camera coordinates

File: cnoid_tank_description/urdf/cnoid_tank.urdf.xacro (robot description, xacro)
@@ -21,5 +21,5 @@
   <link name="Kinect"/>
   <joint name="Kinect" type="fixed">
-    <origin rpy="${M_PI/2} ${M_PI} ${M_PI/2}"/>
+    <origin rpy="${M_PI/2} 0 ${-M_PI/2}"/>
     <parent link="Kinect_base"/>
     <child link="Kinect"/>
